File: kicad/aPortableInductionHeater.kicad_pcb (KiCad board)
At the start: 2 copper layers, 160.3 x 50.8 mm, 27 parts, among them U1 schUCC27211, U2 schUCC27211, U3 schTLV1117-33

Commit message: 2017
Other:
- board text added: "2017 Copyright (C) DELOUCHE-VILPOUX"
- board text removed: "Copyright (C) DELOUCHE-VILPOUX"
Changed lines of the file:
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@@
     (visible_elements FFFFFFFF)
     (pcbplotparams
-      (layerselection 0x010fc_ffffffff)
+      (layerselection 0x010f8_ffffffff)
       (usegerberextensions false)
       (usegerberattributes true)
+      (gerberprecision 5)
       (excludeedgelayer true)
       (linewidth 0.100000)
@@
     )
   )
-  (gr_text "Copyright (C) DELOUCHE-VILPOUX" (at 109.474 132.588) (layer Bottom)
+  (gr_text "2017 Copyright (C) DELOUCHE-VILPOUX" (at 110.998 132.588) (layer Bottom)
     (effects (font (size 1 1) (thickness 0.25)) (justify mirror))
   )
@@
     (effects (font (size 1 1) (thickness 0.25)) (justify mirror))
   )
-  (gr_text "Copyright (C) DELOUCHE-VILPOUX" (at 109.22 129.032) (layer Top)
+  (gr_text "2017 Copyright (C) DELOUCHE-VILPOUX" (at 109.22 129.032) (layer Top)
     (effects (font (size 1 1) (thickness 0.25)))
   )
@@
     (effects (font (size 1 1) (thickness 0.25)))
   )
-  (gr_text "Copyright (C) DELOUCHE-VILPOUX" (at 109.474 132.588) (layer B.SilkS)
+  (gr_text "2017 Copyright (C) DELOUCHE-VILPOUX" (at 110.998 132.588) (layer B.SilkS)
     (effects (font (size 1 1) (thickness 0.25)) (justify mirror))
   )
@@
     (effects (font (size 0.9652 0.9652) (thickness 0.12192)) (justify left bottom))
   )
-  (gr_text "Copyright (C) DELOUCHE-VILPOUX" (at 109.22 129.032) (layer F.SilkS)
+  (gr_text "2017 Copyright (C) DELOUCHE-VILPOUX" (at 109.22 129.032) (layer F.SilkS)
     (effects (font (size 1 1) (thickness 0.25)))
   )
